Commit message: Actualiza el paquete para funcionar conjuntamente con el robot real

File: urdf/modelo_delta.urdf (robot description, URDF)
Before this commit: robot Delta_robot, 13 links, 12 joints
Links:
- link barra1_b: geometry visual box size=0.205 0.02 0.02
- link barra2_b: geometry visual box size=0.205 0.02 0.02
- link barra3_b: geometry visual box size=0.205 0.02 0.02
- link base_link: geometry visual cylinder length=0.05 radius=0.04
- link brazo1: geometry visual box size=0.15 0.03 0.03
- link brazo2: geometry visual box size=0.15 0.03 0.03
- link brazo3: geometry visual box size=0.15 0.03 0.03
Joints:
- joint base_brazo1: origin xyz=0.0620652 0 0 -> xyz=0.0360844 0 0
- joint base_brazo2: origin xyz=-0.0310326 -0.05375 0 rpy=0 0 -2.0944 -> xyz=-0.0180422 -0.03125 0 rpy=0 0 -2.0944
- joint base_brazo3: origin xyz=-0.0310326 0.05375 0 rpy=0 0 2.0944 -> xyz=-0.0180422 0.03125 0 rpy=0 0 2.0944
- joint codo1_a: origin xyz=0.25 0 0 rpy=0 0 0 -> xyz=0.15 0 0 rpy=0 0 0
- joint codo2_a: origin xyz=0.25 0 0 rpy=0 0 0 -> xyz=0.15 0 0 rpy=0 0 0
- joint codo3_a: origin xyz=0.25 0 0 rpy=0 0 0 -> xyz=0.15 0 0 rpy=0 0 0
